Commit message: rtai support, non-uta dependency, xacro styleguide and minor reorganistaion

File: models/xacro/controlit_dreamer.xacro (robot description, xacro)
@@ -2,31 +2,31 @@
 <robot xmlns:xacro="http://ros.org/wiki/xacro" name="dreamer">
     <!-- Define the joint types. This specifies the joints that are controlled by WBOSC. -->
-    <property name="EYE_JOINT_TYPE" value="fixed" />
-    <property name="RIGHT_HAND_JOINT_TYPE" value="fixed" />
-    <property name="LEFT_GRIPPER_JOINT_TYPE" value="fixed" />
-    <property name="JOINT_TYPE_TORSO_YAW"               value="fixed" />
-    <property name="JOINT_TYPE_TORSO_LOWER_PITCH"       value="revolute" />
-    <property name="JOINT_TYPE_TORSO_UPPER_PITCH"       value="revolute" />
-    <property name="JOINT_TYPE_LOWER_NECK_PITCH"        value="fixed" />
-    <property name="JOINT_TYPE_UPPER_NECK_YAW"          value="fixed" />
-    <property name="JOINT_TYPE_UPPER_NECK_ROLL"         value="fixed" />
-    <property name="JOINT_TYPE_UPPER_NECK_PITCH"        value="fixed" />
-    <property name="JOINT_TYPE_LEFT_SHOULDER_EXTENSOR"  value="revolute" />
-    <property name="JOINT_TYPE_LEFT_SHOULDER_ABDUCTOR"  value="revolute" />
-    <property name="JOINT_TYPE_LEFT_SHOULDER_ROTATOR"   value="revolute" />
-    <property name="JOINT_TYPE_LEFT_ELBOW"              value="revolute" />
-    <property name="JOINT_TYPE_LEFT_WRIST_ROTATOR"      value="revolute" />
-    <property name="JOINT_TYPE_LEFT_WRIST_PITCH"        value="revolute" />
-    <property name="JOINT_TYPE_LEFT_WRIST_YAW"          value="revolute" />
-    <property name="JOINT_TYPE_RIGHT_SHOULDER_EXTENSOR" value="revolute" />
-    <property name="JOINT_TYPE_RIGHT_SHOULDER_ABDUCTOR" value="revolute" />
-    <property name="JOINT_TYPE_RIGHT_SHOULDER_ROTATOR"  value="revolute" />
-    <property name="JOINT_TYPE_RIGHT_ELBOW"             value="revolute" />
-    <property name="JOINT_TYPE_RIGHT_WRIST_ROTATOR"     value="revolute" />
-    <property name="JOINT_TYPE_RIGHT_WRIST_PITCH"       value="revolute" />
-    <property name="JOINT_TYPE_RIGHT_WRIST_YAW"         value="revolute" />
+    <xacro:property name="EYE_JOINT_TYPE" value="fixed" />
+    <xacro:property name="RIGHT_HAND_JOINT_TYPE" value="fixed" />
+    <xacro:property name="LEFT_GRIPPER_JOINT_TYPE" value="fixed" />
+    <xacro:property name="JOINT_TYPE_TORSO_YAW"               value="fixed" />
+    <xacro:property name="JOINT_TYPE_TORSO_LOWER_PITCH"       value="revolute" />
+    <xacro:property name="JOINT_TYPE_TORSO_UPPER_PITCH"       value="revolute" />
+    <xacro:property name="JOINT_TYPE_LOWER_NECK_PITCH"        value="fixed" />
+    <xacro:property name="JOINT_TYPE_UPPER_NECK_YAW"          value="fixed" />
+    <xacro:property name="JOINT_TYPE_UPPER_NECK_ROLL"         value="fixed" />
+    <xacro:property name="JOINT_TYPE_UPPER_NECK_PITCH"        value="fixed" />
+    <xacro:property name="JOINT_TYPE_LEFT_SHOULDER_EXTENSOR"  value="revolute" />
+    <xacro:property name="JOINT_TYPE_LEFT_SHOULDER_ABDUCTOR"  value="revolute" />
+    <xacro:property name="JOINT_TYPE_LEFT_SHOULDER_ROTATOR"   value="revolute" />
+    <xacro:property name="JOINT_TYPE_LEFT_ELBOW"              value="revolute" />
+    <xacro:property name="JOINT_TYPE_LEFT_WRIST_ROTATOR"      value="revolute" />
+    <xacro:property name="JOINT_TYPE_LEFT_WRIST_PITCH"        value="revolute" />
+    <xacro:property name="JOINT_TYPE_LEFT_WRIST_YAW"          value="revolute" />
+    <xacro:property name="JOINT_TYPE_RIGHT_SHOULDER_EXTENSOR" value="revolute" />
+    <xacro:property name="JOINT_TYPE_RIGHT_SHOULDER_ABDUCTOR" value="revolute" />
+    <xacro:property name="JOINT_TYPE_RIGHT_SHOULDER_ROTATOR"  value="revolute" />
+    <xacro:property name="JOINT_TYPE_RIGHT_ELBOW"             value="revolute" />
+    <xacro:property name="JOINT_TYPE_RIGHT_WRIST_ROTATOR"     value="revolute" />
+    <xacro:property name="JOINT_TYPE_RIGHT_WRIST_PITCH"       value="revolute" />
+    <xacro:property name="JOINT_TYPE_RIGHT_WRIST_YAW"         value="revolute" />
     <!-- RViz uses package:// for the model path -->
-    <property name="modelPath" value="package://dreamer/models/dreamer" />
-    <property name="gripperModelPath" value="package://dreamer/models/dreamer" />
+    <xacro:property name="modelPath" value="package://dreamer/models/dreamer" />
+    <xacro:property name="gripperModelPath" value="package://dreamer/models/dreamer" />
     <!-- Load the Dreamer Model -->
     <xacro:include filename="$(find dreamer)/models/dreamer/xacro/dreamer_base.xacro" />
